File: TecladoEB.sch (KiCad schematic (older format))
At the start: 11 parts, among them J1 GND-SIG

Commit message: Updated to v1.3, including new LICENSE
Parts:
- J1: value GND-SIG -> Connector; symbol Connector:Conn_01x02 -> Connector:Conn_01x02_Male
- R1, R2, R3, R4: symbol device:R -> Device:R
- R5: value 22k -> 10k; symbol device:R -> Device:R
- S1, S2, S3, S4, S5: symbol EB-B3F-4055:B3F-4055-B3F-4055 -> B3F-4050:B3F-4050
Connections:
- wire segments 32 -> 22
